File: HV-pulse-generator.kicad_pcb (KiCad board)
At the start: 2 copper layers, 235.5 x 99.1 mm, 80 parts, among them J1 CONN_01X03, J2 CONN_01X02, J3 CONN_01X02, J4 CONN_01X02, J5 CONN_01X02, P1 PEM2-S24-S5-S, P2 JCJ0824D15, P3 PEM2-S24-S5-S, P4 JCJ0824D15, Q1 VP0104, Q2 FQP3P50, Q3 VN0104, Q4 VP0104, Q5 FQP13N50, Q6 VN0104, U1 LM7171, U2 ICPL2631, U3 MCP1525, U4 LM7171, U5 LM7171, U6 ICPL2631, U7 MCP1525, U8 LM7171

Commit message: replace first drive transitors
Parts:
- removed CINNEG, CINPOS: 100uF 500V, Capacitors_THT:CP_Radial_D25.0mm_P10.00mm_SnapIn
- removed the REF** at (163.8, 63.8)
- removed the REF** at (191.3, 87.9)
- removed the REF** at (200.2, 128.0)
- removed the REF** at (163.8, 112.0)
- removed the REF** at (250.2, 39.6)
- removed the REF** at (250.2, 131.1)
- removed the REF** at (22.4, 131.1)
- removed the REF** at (22.4, 39.6)
- removed RTUNE: 200, Potentiometers:Potentiometer_Trimmer_Bourns_PV36W
- added C35: 0.01uF, hvhf:C_Disc_D3_P2.5, F.Cu at (72.4, 31.8)
- added C36: 0.1uF, hvhf:C_Disc_D3_P2.5, F.Cu at (66.0, 48.3)
- added C37: 10uF, hvhf:C_Disc_D3_P2.5, F.Cu at (78.7, 58.4)
- added C38: 100uF, hvhf:C_Radial_D6.3_L11.2_P2.5, F.Cu at (33.0, 50.8)
- added REF**: Heatsink_Assmann_V5229x_32x14mm, User_Defined:Heatsink_Assmann_V5229x_32x14mm, F.Cu at (201.9, 76.2)
- added REF**: Heatsink_Assmann_V5229x_32x14mm, User_Defined:Heatsink_Assmann_V5229x_32x14mm, F.Cu at (135.9, 120.7)
- added REF**: Heatsink_Ohmite_R_Series-42x25mm, User_Defined:Heatsink_Ohmite_R_Series-42x25mm, F.Cu at (171.4, 44.5)
- added REF**: Heatsink_Assmann_V5229x_32x14mm, User_Defined:Heatsink_Assmann_V5229x_32x14mm, F.Cu at (228.6, 121.9)
- added REF**: Heatsink_Assmann_V5229x_32x14mm, User_Defined:Heatsink_Assmann_V5229x_32x14mm, F.Cu at (135.9, 94.0)
- added REF**: MountingHole_3.2mm_M3, MountingHole:MountingHole_3.2mm_M3, F.Cu at (25.4, 127.0)
- added REF**: MountingHole_3.2mm_M3, MountingHole:MountingHole_3.2mm_M3, F.Cu at (25.4, 25.4)
- added REF**: MountingHole_3.2mm_M3, MountingHole:MountingHole_3.2mm_M3, F.Cu at (254.0, 25.4)
- added REF**: Heatsink_Ohmite_R_Series-42x25mm, User_Defined:Heatsink_Ohmite_R_Series-42x25mm, F.Cu at (171.4, 108.0)
- added REF**: MountingHole_3.2mm_M3, MountingHole:MountingHole_3.2mm_M3, F.Cu at (254.0, 127.0)
- added REF**: Heatsink_Assmann_V5229x_32x14mm, User_Defined:Heatsink_Assmann_V5229x_32x14mm, F.Cu at (135.9, 57.1)
- added REF**: Heatsink_Assmann_V5229x_32x14mm, User_Defined:Heatsink_Assmann_V5229x_32x14mm, F.Cu at (135.9, 30.5)
- added RTUNE1: 200, Potentiometer_THT:Potentiometer_Bourns_3296W_Vertical, F.Cu at (228.6, 73.7)
- C1: value 2.2uF -> 0.1uF; footprint User_Defined:C_Tantalum_D3_P2.5 -> hvhf:C_Disc_D3_P2.5
- C10: value 0.1uF -> 0.01uF; footprint Capacitors_ThroughHole:C_Disc_D3_P2.5 -> hvhf:C_Disc_D3_P2.5
- C11, C27: value 10uF -> 100uF; footprint Capacitors_ThroughHole:C_Disc_D3_P2.5 -> hvhf:C_Radial_D6.3_L11.2_P2.5
- C12: value 100uF -> 2.2uF; footprint Capacitors_ThroughHole:C_Radial_D6.3_L11.2_P2.5 -> hvhf:C_Tantalum_D3_P2.5
- C13: value 2.2uF -> 1uF; footprint User_Defined:C_Tantalum_D3_P2.5 -> hvhf:C_Disc_D3_P2.5
- C14, C25, C7: footprint Capacitors_ThroughHole:C_Disc_D3_P2.5 -> hvhf:C_Disc_D3_P2.5
- C15: value 1uF -> 100uF; footprint Capacitors_ThroughHole:C_Disc_D3_P2.5 -> hvhf:C_Radial_D6.3_L11.2_P2.5
- C16, C2, C28: value 100uF -> 0.01uF; footprint Capacitors_ThroughHole:C_Radial_D6.3_L11.2_P2.5 -> hvhf:C_Disc_D3_P2.5
- C17: value 100uF -> 0.1uF; footprint Capacitors_ThroughHole:C_Radial_D6.3_L11.2_P2.5 -> hvhf:C_Disc_D3_P2.5
- C18: value 2.2uF -> 10uF; footprint User_Defined:C_Tantalum_D3_P2.5 -> hvhf:C_Disc_D3_P2.5
- C19, C30, C34, C8: footprint Capacitors_ThroughHole:C_Radial_D6.3_L11.2_P2.5 -> hvhf:C_Radial_D6.3_L11.2_P2.5
- C20: value 0.01uF -> 0.1uF; footprint Capacitors_ThroughHole:C_Disc_D3_P2.5 -> hvhf:C_Disc_D3_P2.5
- C21, C33: value 1uF -> 0.01uF; footprint Capacitors_ThroughHole:C_Disc_D3_P2.5 -> hvhf:C_Disc_D3_P2.5
- C22, C26: value 0.1uF -> 100uF; footprint Capacitors_ThroughHole:C_Disc_D3_P2.5 -> hvhf:C_Radial_D6.3_L11.2_P2.5
- C23: value 0.01uF -> 2.2uF; footprint Capacitors_ThroughHole:C_Disc_D3_P2.5 -> hvhf:C_Tantalum_D3_P2.5
- C24: value 100uF -> 1uF; footprint Capacitors_ThroughHole:C_Radial_D6.3_L11.2_P2.5 -> hvhf:C_Disc_D3_P2.5
- C29, C6: footprint User_Defined:ECW-FA2J(10-68)4J -> hvhf:ECW-FA2J(10-68)4J
- C3, C9: value 0.01uF -> 100uF; footprint Capacitors_ThroughHole:C_Disc_D3_P2.5 -> hvhf:C_Radial_D6.3_L11.2_P2.5
- C31: footprint User_Defined:C_Tantalum_D3_P2.5 -> hvhf:C_Tantalum_D3_P2.5
- C32: value 0.01uF -> 1uF; footprint Capacitors_ThroughHole:C_Disc_D3_P2.5 -> hvhf:C_Disc_D3_P2.5
- C4: value 1uF -> 2.2uF; footprint Capacitors_ThroughHole:C_Disc_D3_P2.5 -> hvhf:C_Tantalum_D3_P2.5
- C5: value 0.1uF -> 1uF; footprint Capacitors_ThroughHole:C_Disc_D3_P2.5 -> hvhf:C_Disc_D3_P2.5
- D1, D2: footprint Diodes_ThroughHole:Diode_DO-41_SOD81_Horizontal_RM10 -> hvhf:Diode_DO-41_SOD81_Horizontal_RM10
- J1: footprint User_Defined:Pin_Header_Molex_10-32-1031 -> hvhf:Pin_Header_Molex_10-32-1031
- J2, J5: value CONN_01X02 -> Pin1=TTL Pin2=GND; footprint Pin_Headers:Pin_Header_Straight_1x02 -> Connector_PinHeader_2.54mm:PinHeader_1x02_P2.54mm_Vertical
- J3: value CONN_01X02 -> Pin1=24V Pin2=GND; footprint Pin_Headers:Pin_Header_Straight_1x02 -> Connector_PinHeader_2.54mm:PinHeader_1x02_P2.54mm_Vertical
- J4: footprint User_Defined:Pin_Header_Molex_10-32-1021 -> hvhf:Pin_Header_Molex_10-32-1021
- P1, P3: footprint User_Defined:DCDC-Conv_CUI_PEM2_DUAL -> hvhf:DCDC-Conv_CUI_PEM2_DUAL
- P2, P4: footprint User_Defined:JCJ0824D15 -> hvhf:JCJ0824D15
- Q1, Q4: value VP0104 -> IRF9610PBF; footprint User_Defined:TO92-DGS-VP0104 -> Package_TO_SOT_THT:TO-220-3_Vertical
- Q2: footprint User_Defined:FQP3P20 -> hvhf:FQP3P20
- Q3, Q6: value VN0104 -> IRF710PBF; footprint User_Defined:TO92-DGS-VN0104 -> Package_TO_SOT_THT:TO-220-3_Vertical
- Q5: footprint User_Defined:FQP4N20L -> hvhf:FQP4N20L
- R1, R5, R9: footprint Resistors_ThroughHole:Resistor_TO-220_Vertical -> hvhf:Resistor_TO-220_Vertical
- R2, R3, R6, R7: footprint Resistors_ThroughHole:Resistor_Horizontal_RM7mm -> hvhf:Resistor_Horizontal_RM7mm
- R4, R8: footprint Resistors_ThroughHole:Resistor_Horizontal_RM15mm -> hvhf:Resistor_Horizontal_RM15mm
- U1, U2, U5, U6: footprint Housings_DIP:DIP-8_W7.62mm_LongPads -> Package_DIP:DIP-8_W7.62mm_LongPads
- U3, U7: value MCP1525 -> LM7171; footprint Documents:TO92-MCP1525 -> Package_DIP:DIP-8_W7.62mm_LongPads
- U4, U8: value LM7171 -> MCP1525; footprint Housings_DIP:DIP-8_W7.62mm_LongPads -> hvhf:TO92-MCP1525
- moved C15 115.3 mm to (33.0, 124.5)
- moved C9 102.3 mm to (43.2, 124.5), turned to 0 degrees
- moved C22 95.0 mm to (74.9, 25.4)
- moved C27 89.2 mm to (43.2, 61.0), turned to 0 degrees
- moved C25 87.9 mm to (115.6, 30.5), turned to 270 degrees
- moved C2 87.5 mm to (102.9, 125.7)
- moved P4 84.9 mm to (50.8, 33.0)
- moved C28 77.8 mm to (100.3, 30.5), turned to 270 degrees
- moved C20 76.2 mm to (92.7, 33.0)
- moved U8 76.2 mm to (66.0, 58.4), turned to 90 degrees
- moved C12 75.9 mm to (108.0, 125.8)
- moved C30 75.7 mm to (74.9, 38.1), turned to 270 degrees
- moved U4 75.0 mm to (66.0, 121.9), turned to 90 degrees
- moved C24 74.5 mm to (110.5, 30.5)
- moved C23 74.3 mm to (105.4, 30.5)
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Connections:
- net Net-(J1-Pad3) renamed -VDC
- C1 pad 1: Net-(C1-Pad1) -> /Sheet5F8C1FCD/+5V
- C1 pad 2: Net-(C1-Pad2) -> /Sheet5F8C1FCD/COM
- C10 pad 1: Net-(C10-Pad1) -> /Sheet5F8C1FCD/+15V
- C10 pad 2: Net-(C1-Pad2) -> /Sheet5F8C1FCD/COM
- C11 pad 1: Net-(C11-Pad1) -> /Sheet5F8C1FCD/COM
- C11 pad 2: Net-(C1-Pad2) -> /Sheet5F8C1FCD/-15V
- C12 pad 1: Net-(C12-Pad1) -> /Sheet5F8C1FCD/COM
- C12 pad 2: Net-(C12-Pad2) -> /Sheet5F8C1FCD/-15V
- C13 pad 1: Net-(C1-Pad2) -> /Sheet5F8C1FCD/COM
- C13 pad 2: Net-(C13-Pad2) -> /Sheet5F8C1FCD/-15V
- C14 pad 1: Net-(C13-Pad2) -> /Sheet5F8C1FCD/COM
- C14 pad 2: Net-(C1-Pad2) -> /Sheet5F8C1FCD/-15V
- C15 pad 1: Net-(C13-Pad2) -> +24V
- C15 pad 2: Net-(C1-Pad2) -> GNDPWR
- C16 pad 1: Net-(C1-Pad2) -> /Sheet5F8C1FCD/+15V
- C16 pad 2: Net-(C13-Pad2) -> /Sheet5F8C1FCD/-15V
- C17 pad 1: Net-(C12-Pad1) -> /Sheet5F8C1FCD/+5V
- C17 pad 2: Net-(C12-Pad2) -> /Sheet5F8C1FCD/COM
- C18 pad 1: Net-(C18-Pad1) -> /Sheet5F8C1FCD/+2P5V
- C18 pad 2: Net-(C18-Pad2) -> /Sheet5F8C1FCD/COM
- C19 pad 1: Net-(C18-Pad1) -> +24V
- C19 pad 2: Net-(C18-Pad2) -> GNDPWR
- C2 pad 1: Net-(C1-Pad1) -> /Sheet5F8C1FCD/COM
- C2 pad 2: Net-(C1-Pad2) -> /Sheet5F8C1FCD/-15V
- C20 pad 1: Net-(C18-Pad1) -> /sheet5F874D32/+5V
- C20 pad 2: Net-(C18-Pad2) -> /sheet5F874D32/COM
- C21 pad 1: Net-(C18-Pad1) -> /sheet5F874D32/COM
- C21 pad 2: Net-(C18-Pad2) -> /sheet5F874D32/-15V
- C22 pad 1: Net-(C22-Pad1) -> /sheet5F874D32/+15V
- C22 pad 2: Net-(C18-Pad2) -> /sheet5F874D32/COM
- C23 pad 1: Net-(C23-Pad1) -> /sheet5F874D32/+15V
- C23 pad 2: Net-(C18-Pad2) -> /sheet5F874D32/COM
- C24 pad 1: Net-(C22-Pad1) -> /sheet5F874D32/+15V
- C24 pad 2: Net-(C18-Pad2) -> /sheet5F874D32/COM
- C25 pad 1: Net-(C18-Pad1) -> /sheet5F874D32/+15V
- C25 pad 2: Net-(C18-Pad2) -> /sheet5F874D32/COM
- C26 pad 1: Net-(C22-Pad1) -> /sheet5F874D32/+5V
- C26 pad 2: Net-(C18-Pad2) -> /sheet5F874D32/COM
- C27 pad 1: Net-(C27-Pad1) -> +24V
- C27 pad 2: Net-(C18-Pad2) -> GNDPWR
- C28 pad 1: Net-(C12-Pad1) -> /sheet5F874D32/+15V
- C28 pad 2: Net-(C12-Pad2) -> /sheet5F874D32/COM
- C29 pad 1: Net-(C18-Pad2) -> GND
- C29 pad 2: GND -> /Sheet5F8C1FCD/COM
- C3 pad 1: Net-(C1-Pad1) -> /Sheet5F8C1FCD/+15V
- C3 pad 2: Net-(C1-Pad2) -> /Sheet5F8C1FCD/COM
- C30 pad 1: Net-(C12-Pad1) -> /sheet5F874D32/COM
- C30 pad 2: Net-(C12-Pad2) -> /sheet5F874D32/-15V
- C31 pad 1: Net-(C18-Pad2) -> /sheet5F874D32/COM
- C31 pad 2: Net-(C23-Pad1) -> /sheet5F874D32/-15V
- C32 pad 1: Net-(C23-Pad1) -> /sheet5F874D32/COM
- C32 pad 2: Net-(C18-Pad2) -> /sheet5F874D32/-15V
- C33 pad 1: Net-(C23-Pad1) -> /sheet5F874D32/COM
- C33 pad 2: Net-(C18-Pad2) -> /sheet5F874D32/-15V
- C34 pad 1: Net-(C18-Pad2) -> +24V
- C34 pad 2: Net-(C23-Pad1) -> GNDPWR
- C4 pad 1: Net-(C1-Pad1) -> /Sheet5F8C1FCD/+15V
- C4 pad 2: Net-(C1-Pad2) -> /Sheet5F8C1FCD/COM
- C5 pad 1: Net-(C10-Pad1) -> /Sheet5F8C1FCD/+15V
- C5 pad 2: Net-(C1-Pad2) -> /Sheet5F8C1FCD/COM
- C6 pad 1: Net-(C1-Pad2) -> /sheet5F874D32/COM
- C7 pad 1: Net-(C13-Pad2) -> /Sheet5F8C1FCD/+15V
- C7 pad 2: Net-(C1-Pad2) -> /Sheet5F8C1FCD/COM
- C8 pad 1: Net-(C10-Pad1) -> /Sheet5F8C1FCD/+5V
- C8 pad 2: Net-(C1-Pad2) -> /Sheet5F8C1FCD/COM
- C9 pad 1: Net-(C1-Pad1) -> +24V
- C9 pad 2: Net-(C1-Pad2) -> GNDPWR
- D1 pad 2: Net-(D1-Pad2) -> /Sheet5F8C1FCD/GATE
- D2 pad 2: Net-(D2-Pad2) -> /sheet5F874D32/GATE
- J1 pad 1: Net-(J1-Pad1) -> +VDC
- J2 pad 1: Net-(J2-Pad1) -> /sheet5F874D32/TTL+
- J2 pad 2: Net-(J2-Pad2) -> /sheet5F874D32/TTL-
- J3 pad 1: Net-(C12-Pad1) -> +24V
- J3 pad 2: Net-(C12-Pad2) -> GNDPWR
- J5 pad 1: Net-(J5-Pad1) -> /Sheet5F8C1FCD/TTL+
- J5 pad 2: Net-(J5-Pad2) -> /Sheet5F8C1FCD/TTL-
- P1 pad 1: Net-(C12-Pad1) -> +24V
- P1 pad 2: Net-(C12-Pad2) -> GNDPWR
- P1 pad 5: Net-(C1-Pad2) -> /Sheet5F8C1FCD/COM
- P1 pad 7: Net-(C10-Pad1) -> /Sheet5F8C1FCD/+5V
- P2 pad 11: Net-(C13-Pad2) -> /Sheet5F8C1FCD/-15V
- P2 pad 14: Net-(C1-Pad1) -> /Sheet5F8C1FCD/+15V
- P2 pad 16: Net-(C1-Pad2) -> /Sheet5F8C1FCD/COM
- P2 pad 2: Net-(C12-Pad2) -> GNDPWR
- P2 pad 22: Net-(C12-Pad1) -> +24V
- P2 pad 23: Net-(C12-Pad1) -> +24V
- P2 pad 3: Net-(C12-Pad2) -> GNDPWR
- P2 pad 9: Net-(C1-Pad2) -> /Sheet5F8C1FCD/COM
- P3 pad 1: Net-(C12-Pad1) -> +24V
- P3 pad 2: Net-(C12-Pad2) -> GNDPWR
- P3 pad 5: Net-(C18-Pad2) -> /sheet5F874D32/COM
- P3 pad 7: Net-(C22-Pad1) -> /sheet5F874D32/+5V
- P4 pad 11: Net-(C23-Pad1) -> /sheet5F874D32/-15V
- P4 pad 14: Net-(C18-Pad1) -> /sheet5F874D32/+15V
- P4 pad 16: Net-(C18-Pad2) -> /sheet5F874D32/COM
- P4 pad 2: Net-(C12-Pad2) -> GNDPWR
- P4 pad 22: Net-(C12-Pad1) -> +24V
- P4 pad 23: Net-(C12-Pad1) -> +24V
- P4 pad 3: Net-(C12-Pad2) -> GNDPWR
- P4 pad 9: Net-(C18-Pad2) -> /sheet5F874D32/COM
- Q1 pad 1: Net-(D1-Pad2) -> Net-(Q1-Pad1)
- Q1 pad 2: Net-(Q1-Pad2) -> Net-(D1-Pad1)
- Q1 pad 3: Net-(C1-Pad1) -> /Sheet5F8C1FCD/+15V
- Q2 pad 1: Net-(C1-Pad2) -> /sheet5F874D32/COM
- Q2 pad 3: Net-(D1-Pad1) -> /sheet5F874D32/GATE
- Q3 pad 1: Net-(D1-Pad2) -> Net-(Q3-Pad1)
- Q3 pad 2: Net-(Q3-Pad2) -> Net-(D1-Pad1)
- Q3 pad 3: Net-(C13-Pad2) -> /Sheet5F8C1FCD/-15V
- Q4 pad 1: Net-(D2-Pad1) -> Net-(Q4-Pad1)
- Q4 pad 2: Net-(Q4-Pad2) -> Net-(D2-Pad1)
- Q4 pad 3: Net-(C18-Pad1) -> /sheet5F874D32/+15V
- Q5 pad 1: Net-(C18-Pad2) -> /Sheet5F8C1FCD/COM
- Q5 pad 3: Net-(D2-Pad2) -> /Sheet5F8C1FCD/GATE
- Q6 pad 1: Net-(D2-Pad1) -> Net-(Q6-Pad1)
- Q6 pad 2: Net-(Q6-Pad2) -> Net-(D2-Pad1)
- Q6 pad 3: Net-(C23-Pad1) -> /sheet5F874D32/-15V
- R1 pad 1: Net-(J1-Pad1) -> /sheet5F874D32/COM
- R1 pad 2: Net-(C1-Pad2) -> +VDC
- R2 pad 2: Net-(C10-Pad1) -> /Sheet5F8C1FCD/+5V
- R3 pad 2: Net-(J2-Pad1) -> /Sheet5F8C1FCD/TTL+
- R4 pad 1: Net-(D1-Pad1) -> /Sheet5F8C1FCD/GATE
- R4 pad 2: Net-(D1-Pad2) -> Net-(D1-Pad1)
- R5 pad 1: Net-(J4-Pad1) -> Net-(R5-Pad1)
- R6 pad 2: Net-(C22-Pad1) -> /sheet5F874D32/+5V
- R7 pad 2: Net-(J5-Pad1) -> /sheet5F874D32/TTL+
- R8 pad 1: Net-(D2-Pad2) -> /sheet5F874D32/GATE
- R9 pad 2: Net-(C18-Pad2) -> /Sheet5F8C1FCD/COM
- U1 pad 3: Net-(C11-Pad1) -> /Sheet5F8C1FCD/+2P5V
- U1 pad 4: Net-(C13-Pad2) -> /Sheet5F8C1FCD/-15V
- U1 pad 6: Net-(Q1-Pad2) -> Net-(Q1-Pad1)
- U1 pad 7: Net-(C1-Pad1) -> /Sheet5F8C1FCD/+15V
- U2 pad 2: Net-(J2-Pad2) -> /Sheet5F8C1FCD/TTL-
- U2 pad 5: Net-(C1-Pad2) -> /Sheet5F8C1FCD/COM
- U2 pad 8: Net-(C10-Pad1) -> /Sheet5F8C1FCD/+5V
- U3 pad 1: Net-(C10-Pad1) -> (no net)
- U3 pad 2: Net-(C11-Pad1) -> Net-(R2-Pad1)
- U3 pad 3: Net-(C1-Pad2) -> /Sheet5F8C1FCD/+2P5V
- U4 pad 1: (no net) -> /Sheet5F8C1FCD/+5V
- U4 pad 2: Net-(R2-Pad1) -> /Sheet5F8C1FCD/+2P5V
- U4 pad 3: Net-(C11-Pad1) -> /Sheet5F8C1FCD/COM
- U5 pad 3: Net-(C27-Pad1) -> /sheet5F874D32/+2P5V
- U5 pad 4: Net-(C23-Pad1) -> /sheet5F874D32/-15V
- U5 pad 6: Net-(Q4-Pad2) -> Net-(Q4-Pad1)
- U5 pad 7: Net-(C18-Pad1) -> /sheet5F874D32/+15V
- U6 pad 2: Net-(J5-Pad2) -> /sheet5F874D32/TTL-
- U6 pad 5: Net-(C18-Pad2) -> /sheet5F874D32/COM
- U6 pad 8: Net-(C22-Pad1) -> /sheet5F874D32/+5V
- U7 pad 1: Net-(C22-Pad1) -> (no net)
- U7 pad 2: Net-(C27-Pad1) -> Net-(R6-Pad1)
- U7 pad 3: Net-(C18-Pad2) -> /sheet5F874D32/+2P5V
- U8 pad 1: (no net) -> /sheet5F874D32/+5V
- U8 pad 2: Net-(R6-Pad1) -> /sheet5F874D32/+2P5V
- U8 pad 3: Net-(C27-Pad1) -> /sheet5F874D32/COM
Routing:
- net Net-(C1-Pad2): track 278.0 -> 0.00 mm
- net Net-(C18-Pad2): track 215.4 -> 0.00 mm
- net /sheet5F874D32/-15V: track 0.00 -> 142.4 mm
- net Net-(C22-Pad1): track 104.2 -> 0.00 mm
- net Net-(Q2-Pad2): track 17.8 -> 115.2 mm
- net Net-(C10-Pad1): track 96.7 -> 0.00 mm
- net /Sheet5F8C1FCD/-15V: track 0.00 -> 81.1 mm
- net /sheet5F874D32/+5V: track 0.00 -> 73.9 mm
- net /Sheet5F8C1FCD/+5V: track 0.00 -> 71.2 mm
- net -VDC: track 0.00 -> 60.8 mm
- net /sheet5F874D32/+2P5V: track 0.00 -> 53.1 mm
- net /Sheet5F8C1FCD/+2P5V: track 0.00 -> 53.1 mm
- net Net-(C13-Pad2): track 50.2 -> 0.00 mm
- net Net-(C1-Pad1): track 48.9 -> 0.00 mm
- net GND: track 14.5 -> 63.4 mm
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- added copper zone on B.Cu, net +24V
- added copper zone on B.Cu, net /Sheet5F8C1FCD/+15V
- added copper zone on B.Cu, net /Sheet5F8C1FCD/-15V
- added copper zone on F.Cu, net /Sheet5F8C1FCD/COM
- added copper zone on B.Cu, net /sheet5F874D32/+15V
- added copper zone on B.Cu, net /sheet5F874D32/-15V
- added copper zone on F.Cu, net /sheet5F874D32/COM
- added copper zone on F.Cu, net GND
- added copper zone on F.Cu, net GNDPWR
- removed copper zone on F.Cu, net -VDC
- removed copper zone on B.Cu, net GND
- removed copper zone on B.Cu, net Net-(C1-Pad1)
- removed copper zone on F.Cu, net Net-(C1-Pad2)
- removed copper zone on B.Cu, net Net-(C12-Pad1)
- removed copper zone on F.Cu, net Net-(C12-Pad2)
- removed copper zone on B.Cu, net Net-(C13-Pad2)
- removed copper zone on B.Cu, net Net-(C18-Pad1)
- removed copper zone on B.Cu, net Net-(C18-Pad2)
- removed copper zone on F.Cu, net Net-(C18-Pad2)
- removed copper zone on B.Cu, net Net-(C23-Pad1)
- removed copper zone on F.Cu, net Net-(J1-Pad1)
- removed copper zone on B.Cu, net Net-(J4-Pad1)
- removed copper zone on F.Cu, net Net-(J4-Pad1)
- removed copper zone on B.Cu, net Net-(Q2-Pad2)
Other:
- board size 235.5 x 99.1 mm -> 238.8 x 111.8 mm
- net class Default: clearance 0.2 -> 0.254; trace_width 0.25 -> 0.762
- net class Interal-driving: clearance 0.381 -> 0.254; trace_width 0.4572 -> 0.762
- net class Output: clearance 0.762 -> 0.254; trace_width 0.889 -> 0.762
- rule trace_clearance: 0.2 -> 0.254
- board text added: "+"
- board text added: "+24 V IN"
- board text added: "-"
- board text added: "GND"
- board text added: "NEG DRIVER"
- board text added: "OUT"
- board text added: "POS DRIVER"
- board text removed: "500 V Pulse Generating Board Designed By: Nathan M. Hoffman"
- board text removed: "Peter T.A. Reilly Group Washington State University"

Commit message: 2.0.0
Parts:
- removed J1: CONN_01X03, hvhf:Pin_Header_Molex_10-32-1031
- added J1.1: Pin1=24V Pin2=GND, Connector_PinHeader_2.54mm:PinHeader_1x02_P2.54mm_Vertical, F.Cu at (247.7, 64.8)
- added J1.2: Pin1=24V Pin2=GND, Connector_PinHeader_2.54mm:PinHeader_1x02_P2.54mm_Vertical, F.Cu at (247.7, 90.2)
- J4: footprint hvhf:Pin_Header_Molex_10-32-1021 -> Connector_PinHeader_2.54mm:PinHeader_1x02_P2.54mm_Vertical
- moved REF** 27.4 mm to (201.9, 115.6), turned to 90 degrees
- moved REF** 27.4 mm to (201.9, 36.8), turned to 90 degrees
- moved R1 25.9 mm to (203.2, 36.8), turned to 90 degrees
- moved R9 25.9 mm to (203.2, 115.6), turned to 90 degrees
- moved R8 15.2 mm to (143.5, 43.2), turned to 0 degrees
- moved J4 14.0 mm to (247.7, 77.5)
- moved D2 10.2 mm to (158.8, 48.3), turned to 180 degrees
Connections:
- D1 pad 1: Net-(D1-Pad1) -> /Sheet5F8C1FCD/GATE
- D1 pad 2: /Sheet5F8C1FCD/GATE -> Net-(D1-Pad2)
- Q1 pad 2: Net-(D1-Pad1) -> /Sheet5F8C1FCD/GATE
- Q2 pad 3: /sheet5F874D32/GATE -> Net-(D2-Pad1)
- Q3 pad 2: Net-(D1-Pad1) -> /Sheet5F8C1FCD/GATE
- Q4 pad 2: Net-(D2-Pad1) -> /sheet5F874D32/GATE
- Q5 pad 3: /Sheet5F8C1FCD/GATE -> Net-(D1-Pad2)
- Q6 pad 2: Net-(D2-Pad1) -> /sheet5F874D32/GATE
- R4 pad 1: /Sheet5F8C1FCD/GATE -> Net-(D1-Pad2)
- R4 pad 2: Net-(D1-Pad1) -> /Sheet5F8C1FCD/GATE
- RTUNE1 pad 1: Net-(J4-Pad1) -> (no net)
- RTUNE1 pad 3: Net-(R5-Pad1) -> Net-(J4-Pad1)
Routing:
- net Net-(D1-Pad1): track 47.2 -> 0.00 mm
- net /Sheet5F8C1FCD/GATE: track 15.8 -> 47.2 mm
- net Net-(D2-Pad1): track 47.2 -> 15.8 mm
- net /sheet5F874D32/GATE: track 15.8 -> 47.2 mm
- net +VDC: track 38.2 -> 68.7 mm
- net -VDC: track 60.8 -> 78.7 mm
- net Net-(D1-Pad2): track 0.00 -> 15.8 mm
- net GND: track 63.4 -> 76.6 mm
- net Net-(J4-Pad1): track 30.9 -> 19.6 mm
- net Net-(R5-Pad1): track 27.9 -> 26.5 mm
Other:
- board text added: "HIGH VOLTAGE"
- board text added: "HIGH VOLTAGE PULSE GENERATOR VERSION 2.0.0 SEPTEMBER 2020"
- board text added: "NEG"
- board text added: "POS"

Commit message: initial commit
Other:
- net class Default removed
- net class Interal-driving removed
- net class Output removed
